File: Combined-MCU-GPS-LoRa/gps.kicad_sch (KiCad schematic)
At the start: 0 parts

Commit message: Added Readme
Parts:
- added C1: 10uF, Capacitor_SMD:C_0402_1005Metric, symbol Device:C
- added C2: 100nF, Capacitor_SMD:C_1206_3216Metric, symbol Device:C
- added C3: 470pF, Capacitor_SMD:C_1206_3216Metric, symbol Device:C
- added L1: 6.8nH, Inductor_SMD:L_0402_1005Metric, symbol Device:L
- added R1: 1k, symbol Device:R
- added U1: ATGM336H-5N31, PARTS:RA_08H-BREAKOUT, symbol PARTS:ATGM336H-5N31
- added U2: AT2659, PARTS:AT2659, symbol PARTS:AT2659
- added U4: BWU.FL-IPEX1, PARTS:IPEX-SMD_BWIPX-1-001E, symbol PARTS:BWU.FL-IPEX1
Connections:
- new net: C3.1, L1.2
- new net: C3.2, U4.1
- new net: U1.11 (RF_IN), U2.6 (RFOUT)
- new net: R1.1, U1.14 (VCC_RF)
- new net: L1.1, U2.3 (RFIN)
- new net 1PPS: U1.4 (1PPS)
- new net 3v3_GPS: C1.1, C2.1, U1.8 (VCC), U2.4 (VDD), U2.5 (/SHDN)
- new net GND: C1.2, C2.2, R1.2, U1.1 (GND), U1.10 (GND), U1.12 (GND), U2.1 (GND), U2.2 (GND), U4.2, U4.3
- new net ON_OFF: U1.5 (ON/OFF)
- new net RST: U1.9 (NRESET)
- new net RXD: U1.3 (RXD)
- new net SCL: U1.17 (SCL)
- new net SDA: U1.16 (SDA)
- new net TXD: U1.2 (TXD)
- new net VBAT: U1.6 (VBAT)
- no-connect marks 0 -> 5
