File: Combined-MCU-GPS-LoRa/lora.kicad_sch (KiCad schematic)
At the start: 0 parts

Commit message: Added Readme
Parts:
- added C3: 0.1uF, Capacitor_SMD:C_1206_3216Metric, symbol Device:C
- added C4: 10uF, Capacitor_SMD:C_0402_1005Metric, symbol Device:C
- added D1, D2: D_Schottky, Diode_SMD:D_SMA, symbol Device:D_Schottky
- added U1: RA-08H(915), PARTS:RA_08H-BREAKOUT, symbol PARTS:RA-08H(915)
- added U2: BWU.FL-IPEX1, PARTS:IPEX-SMD_BWIPX-1-001E, symbol PARTS:BWU.FL-IPEX1
Connections:
- new net: U1.18 (ANT), U2.1
- new net: D1.2 (A), D2.2 (A)
- new net 3v3_LORA: C3.1, C4.1, D1.1 (K), U1.9 (VCC)
- new net GND: C3.2, C4.2, D2.1 (K), U1.1 (GND), U1.17 (GND), U2.2, U2.3
- new net LPRXD: U1.10 (LPRXD)
- new net RST: U1.16 (RST)
- new net TXD: U1.11 (TXD)
- no-connect marks 0 -> 11
