File: Combined/Combined.kicad_sch (KiCad schematic)
At the start: 4 parts, among them U1 ATMEGA168PA-MU, U2 RA-08H(915), U3 ATGM336H-5N31, U4 X1B000301000200

Commit message: Working on combined schematic.
Parts:
- added C1, C2, C3, C4, C5, C6: 10u, Capacitor_SMD:C_0402_1005Metric, symbol Device:C
- added U5, U6, U7: ~, Package_TO_SOT_SMD:SOT-23-5, symbol PARTS:MT9700
- U1: footprint PARTS:VQFN-32_L5.0-W5.0-P0.50-TL-EP -> PARTS:168P_BOARD; LCSC Part C1337182 -> (none)
- U2: footprint PARTS:COMM-SMD_18P-L16.0-W16.0-P1.27-BL_RA-08H -> PARTS:RA_08H-BREAKOUT; LCSC Part C2991932 -> (none)
- U3: footprint PARTS:GPSM-SMD_ATGM336H-TR -> PARTS:GPS_BOARD; LCSC Part C90770 -> (none)
- U4: footprint PARTS:OSC-SMD_10P-L3.2-W2.5-BL-1 -> PARTS:RTC_BOARD; LCSC Part C7528386 -> (none)
Connections:
- net GND: now also C1.2, C2.2, C3.2, C4.2, C5.2, C6.2, U5.2 (GND), U6.2 (GND), U7.2 (GND)
- net GPS_I/O: now also U1.11 ((PCINT23/AIN1)PD7)
- net GPS_RESET: now also U1.10 ((PCINT22/OC0A/AIN0)PD6)
- net LoRa_RST: now also U1.9 ((PCINT21/OC0B/T1)PD5)
- net VBAT: now also U1.19 (ADC6)
- net VCC: now also C2.1, C4.1, C6.1, U5.5 (VIN), U6.5 (VIN), U7.5 (VIN); no longer U2.9 (VCC), U3.8 (VCC), U4.2 (VDD)
- net RTC_EN: now reaches U1.12 ((PCINT0/CLKO/ICP1)PB0)
- net RTC_EN: now also U7.4 (EN)
- net LORA_EN: now reaches U1.13 ((PCINT1/OC1A)PB1)
- net LORA_EN: now also U6.4 (EN)
- net GPS_EN: now reaches U1.14 ((PCINT2/SS/OC1B)PB2)
- net GPS_EN: now also U5.4 (EN)
- new net GPS_VCC: C1.1, U3.8 (VCC), U5.1 (VOUT)
- new net LORA_VCC: C3.1, U2.9 (VCC), U6.1 (VOUT)
- new net RTC_VCC: C5.1, U4.2 (VDD), U7.1 (VOUT)
- no-connect marks 24 -> 26
Other:
- note added: "GPS S/W"
- note added: "Lora S/W"
- note added: "RTC S/W"

Commit message: Working.
Parts:
- added BT1: RJD2048(Bat), Connector_PinHeader_2.54mm:PinHeader_1x02_P2.54mm_Vertical, symbol Device:Battery_Cell
- added C7: 100n, symbol Device:C
- added Q1, Q2: 2N7002E, Package_TO_SOT_SMD:SOT-23, symbol Transistor_FET:2N7002E
- added R1: 0.01, Resistor_SMD:R_0805_2012Metric, symbol Device:R
- added R2: 330, symbol Device:R
- added R3: 2.7k, symbol Device:R
- added SC1: KXOB081K06TF-TR, Connector_PinHeader_2.54mm:PinHeader_1x02_P2.54mm_Vertical, symbol Device:Solar_Cell
- added U9: AP9101CK-AHTRG1, PARTS:SOT-23-5_L3.0-W1.7-P0.95-LS2.8-BL, symbol PARTS:AP9101C
Connections:
- net VBAT is gone; now on net VCC: U1.19 (ADC6), U3.6 (VBAT), U4.3 (VBAT)
- net GND: now also C7.2, Q1.2 (S), R1.2, U9.3 (VSS)
- net VCC: now also BT1.1 (+), R2.1, SC1.1 (+)
- net VBAT_SNS: now reaches U1.22 (ADC7)
- net VBAT_SNS: now also BT1.2 (-), R1.1
- new net: C7.1, R2.2, U9.2 (VDD)
- new net: Q2.1 (G), U9.5 (CO)
- new net: Q1.3 (D), Q2.3 (D)
- new net: Q1.1 (G), U9.4 (DO)
- new net: R3.1, U9.1 (VM)
- new net P-: Q2.2 (S), R3.2, SC1.2 (-)
Other:
- moved on the sheet: C1, C2, C3, C4, C5, C6, U1, U5, U6, U7
