File: gen/gen.kicad_pcb (KiCad board)
At the start: 2 copper layers, 40.6 x 40.6 mm, 16 parts

Commit message: Connections
Parts:
- added J1: Conn_01x02_Pin, Connector_PinHeader_2.54mm:PinHeader_1x02_P2.54mm_Vertical, F.Cu at (152.5, 93.1)
- CL1, CL10, CL11, CL12, CL13, CL14, CL15, CL16, CL2, CL3, CL4, CL5, CL6, CL7, CL8, CL9: value SMALL_COIL -> L
Connections:
- CL1 pad 1: (no net) -> Net-(J1-Pin_1)
- CL1 pad 2: (no net) -> Net-(CL1-Pad2)
- CL10 pad 1: (no net) -> Net-(CL10-Pad1)
- CL10 pad 2: (no net) -> Net-(CL10-Pad2)
- CL11 pad 1: (no net) -> Net-(CL10-Pad2)
- CL11 pad 2: (no net) -> Net-(CL11-Pad2)
- CL12 pad 1: (no net) -> Net-(CL11-Pad2)
- CL12 pad 2: (no net) -> Net-(CL12-Pad2)
- CL13 pad 1: (no net) -> Net-(CL12-Pad2)
- CL13 pad 2: (no net) -> Net-(CL13-Pad2)
- CL14 pad 1: (no net) -> Net-(CL13-Pad2)
- CL14 pad 2: (no net) -> Net-(CL14-Pad2)
- CL15 pad 1: (no net) -> Net-(CL14-Pad2)
- CL15 pad 2: (no net) -> Net-(CL15-Pad2)
- CL16 pad 1: (no net) -> Net-(CL15-Pad2)
- CL16 pad 2: (no net) -> Net-(J1-Pin_2)
- CL2 pad 1: (no net) -> Net-(CL1-Pad2)
- CL2 pad 2: (no net) -> Net-(CL2-Pad2)
- CL3 pad 1: (no net) -> Net-(CL2-Pad2)
- CL3 pad 2: (no net) -> Net-(CL3-Pad2)
- CL4 pad 1: (no net) -> Net-(CL3-Pad2)
- CL4 pad 2: (no net) -> Net-(CL4-Pad2)
- CL5 pad 1: (no net) -> Net-(CL4-Pad2)
- CL5 pad 2: (no net) -> Net-(CL5-Pad2)
- CL6 pad 1: (no net) -> Net-(CL5-Pad2)
- CL6 pad 2: (no net) -> Net-(CL6-Pad2)
- CL7 pad 1: (no net) -> Net-(CL6-Pad2)
- CL7 pad 2: (no net) -> Net-(CL7-Pad2)
- CL8 pad 1: (no net) -> Net-(CL7-Pad2)
- CL8 pad 2: (no net) -> Net-(CL8-Pad2)
- CL9 pad 1: (no net) -> Net-(CL8-Pad2)
- CL9 pad 2: (no net) -> Net-(CL10-Pad1)
Routing:
- net Net-(CL6-Pad2): track 0.00 -> 4.95 mm, vias 0 -> 2
- net Net-(J1-Pin_1): track 0.00 -> 4.30 mm
- net Net-(J1-Pin_2): track 0.00 -> 3.84 mm
- net Net-(CL13-Pad2): track 0.00 -> 3.71 mm, vias 0 -> 2
- net Net-(CL10-Pad1): track 0.00 -> 3.43 mm, vias 0 -> 2
- net Net-(CL4-Pad2): track 0.00 -> 3.43 mm, vias 0 -> 2
- net Net-(CL7-Pad2): track 0.00 -> 3.36 mm, vias 0 -> 2
- net Net-(CL2-Pad2): track 0.00 -> 3.36 mm, vias 0 -> 2
- net Net-(CL11-Pad2): track 0.00 -> 3.36 mm, vias 0 -> 2
- net Net-(CL1-Pad2): track 0.00 -> 3.04 mm, vias 0 -> 2
- net Net-(CL8-Pad2): track 0.00 -> 3.04 mm, vias 0 -> 2
- net Net-(CL12-Pad2): track 0.00 -> 3.04 mm, vias 0 -> 2
- net Net-(CL3-Pad2): track 0.00 -> 2.97 mm, vias 0 -> 2
- net Net-(CL14-Pad2): track 0.00 -> 2.97 mm, vias 0 -> 2
- net Net-(CL15-Pad2): track 0.00 -> 2.97 mm, vias 0 -> 2
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Other:
- board text added: "COILS 2"
