File: gen/gen.kicad_sch (KiCad schematic)
At the start: 16 parts

Commit message: Made Connections
Parts:
- added J1: Conn_01x02_Pin, symbol Connector:Conn_01x02_Pin
Connections:
- net at CL5.1: now also CL4.2
- net at CL5.2: now also CL6.1
- net at CL14.1: now also CL13.2
- net at CL14.2: now also CL15.1
- net at CL15.2: now also CL16.1
- net at CL7.1: now also CL6.2
- net at CL7.2: now also CL8.1
- net at CL2.1: now also CL1.2
- net at CL2.2: now also CL3.1
- net at CL12.1: now also CL11.2
- net at CL12.2: now also CL13.1
- net at CL1.1: now also J1.1 (Pin_1)
- net at CL3.2: now also CL4.1
- net at CL9.1: now also CL8.2
- net at CL9.2: now also CL10.1
- net at CL10.2: now also CL11.1
- net at CL16.2: now also J1.2 (Pin_2)
Other:
- moved on the sheet: CL1, CL10, CL11, CL12, CL13, CL14, CL15, CL16, CL2, CL3, CL4, CL5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

Commit message: Connections
Parts:
- CL1, CL10, CL11, CL12, CL13, CL14, CL15, CL16, CL2, CL3, CL4, CL5, CL6, CL7, CL8, CL9: footprint (none) -> PCB Coils:SMALL_COIL
- J1: footprint (none) -> Connector_PinHeader_2.54mm:PinHeader_1x02_P2.54mm_Vertical
Changed lines of the file:
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@@
 			)
 		)
-		(property "Footprint" ""
+		(property "Footprint" "PCB Coils:SMALL_COIL"
 			(at 137.16 62.23 0)
 			(effects
@@
 			)
 		)
-		(property "Footprint" ""
+		(property "Footprint" "Connector_PinHeader_2.54mm:PinHeader_1x02_P2.54mm_Vertical"
 			(at 80.01 81.28 0)
 			(effects
@@
 			)
 		)
-		(property "Footprint" ""
+		(property "Footprint" "PCB Coils:SMALL_COIL"
 			(at 137.16 130.81 0)
 			(effects
@@
 			)
 		)
-		(property "Footprint" ""
+		(property "Footprint" "PCB Coils:SMALL_COIL"
 			(at 137.16 138.43 0)
 			(effects
@@
 			)
 		)
-		(property "Footprint" ""
+		(property "Footprint" "PCB Coils:SMALL_COIL"
 			(at 137.16 77.47 0)
 			(effects
@@
 			)
 		)
-		(property "Footprint" ""
+		(property "Footprint" "PCB Coils:SMALL_COIL"
 			(at 137.16 39.37 0)
 			(effects
@@
 			)
 		)
-		(property "Footprint" ""
+		(property "Footprint" "PCB Coils:SMALL_COIL"
 			(at 137.16 115.57 0)
 			(effects
@@
 			)
 		)
-		(property "Footprint" ""
+		(property "Footprint" "PCB Coils:SMALL_COIL"
 			(at 137.16 123.19 0)
 			(effects
@@
 			)
 		)
-		(property "Footprint" ""
+		(property "Footprint" "PCB Coils:SMALL_COIL"
 			(at 137.16 31.75 0)
 			(effects
@@
 			)
 		)
-		(property "Footprint" ""
+		(property "Footprint" "PCB Coils:SMALL_COIL"
 			(at 137.16 46.99 0)
 			(effects
@@
 			)
 		)
-		(property "Footprint" ""
+		(property "Footprint" "PCB Coils:SMALL_COIL"
 			(at 137.16 92.71 0)
 			(effects
@@
 			)
 		)
-		(property "Footprint" ""
+		(property "Footprint" "PCB Coils:SMALL_COIL"
 			(at 137.16 85.09 0)
 			(effects
@@
 			)
 		)
-		(property "Footprint" ""
+		(property "Footprint" "PCB Coils:SMALL_COIL"
 			(at 137.16 54.61 0)
 			(effects
@@
 			)
 		)
-		(property "Footprint" ""
+		(property "Footprint" "PCB Coils:SMALL_COIL"
 			(at 137.16 100.33 0)
 			(effects
@@
 			)
 		)
-		(property "Footprint" ""
+		(property "Footprint" "PCB Coils:SMALL_COIL"
 			(at 137.16 107.95 0)
 			(effects
@@
 			)
 		)
-		(property "Footprint" ""
+		(property "Footprint" "PCB Coils:SMALL_COIL"
 			(at 137.16 69.85 0)
 			(effects
@@
 			)
 		)
-		(property "Footprint" ""
+		(property "Footprint" "PCB Coils:SMALL_COIL"
 			(at 137.16 146.05 0)
 			(effects
